File: PCB/Clavis.kicad_pcb (KiCad board)
At the start: 2 copper layers, 330 x 108.5 mm, 130 parts, among them SW1 SW_Push, SW10 SW_Push, SW11 SW_Push, SW12 SW_Push, SW13 SW_Push, SW14 SW_Push, SW15 SW_Push, SW16 SW_Push, SW17 SW_Push, SW18 SW_Push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

Commit message: changed a few things
Parts:
- added G***: LOGO, logos:clavis_30x30mm, F.Cu at (346.4, 158.2)
- added G***: LOGO, logos:rudransh, B.Cu at (343.5, 157.3)
